File: THIRD_MIXER_sch.kicad_sch (KiCad schematic)
At the start: 4 parts, among them U2201 ADE-1

Commit message: Update pcb database to version 6
Parts:
- R2201: symbol Custom:R_US_0805_1%_HS -> custom:R_US_0805_1%_HS; PartNumber 800235-180 -> 800235-XXX
- R2202, R2203: symbol Custom:R_US_0805_1%_HS -> custom:R_US_0805_1%_HS; PartNumber 800235-301 -> 800235-XXX
- U2201: symbol Custom:ADE-1 -> custom:ADE-1
Changed lines of the file:
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@@
     (effects (font (size 1.27 1.27)) (justify right))
   )
-  (symbol (lib_id "Custom:ADE-1") (at 147.32 88.9 0)
+  (symbol (lib_id "custom:ADE-1") (at 147.32 88.9 0) (unit 1)
     (in_bom yes) (on_board yes)
     (property "Reference" "U2201" (id 0) (at 138.43 80.01 0)
@@
     (pin "6")
   )
-  (symbol (lib_id "Custom:GND_US") (at 116.84 73.66 0)
+  (symbol (lib_id "custom:GND_US") (at 116.84 73.66 0) (unit 1)
     (in_bom yes) (on_board yes)
     (property "Reference" "#PWR02202" (id 0) (at 116.332 76.962 0)
@@
     (pin "1")
   )
-  (symbol (lib_id "Custom:GND_US") (at 147.32 102.87 0)
+  (symbol (lib_id "custom:GND_US") (at 147.32 102.87 0) (unit 1)
     (in_bom yes) (on_board yes)
     (property "Reference" "#PWR02204" (id 0) (at 146.812 106.172 0)
@@
     (pin "1")
   )
-  (symbol (lib_id "Custom:GND_US") (at 151.13 102.87 0)
+  (symbol (lib_id "custom:GND_US") (at 151.13 102.87 0) (unit 1)
     (in_bom yes) (on_board yes)
     (property "Reference" "#PWR02205" (id 0) (at 150.622 106.172 0)
@@
     (pin "1")
   )
-  (symbol (lib_id "Custom:R_US_0805_1%_HS") (at 100.33 68.58 0)
+  (symbol (lib_id "custom:R_US_0805_1%_HS") (at 100.33 68.58 0) (unit 1)
     (in_bom yes) (on_board yes)
     (property "Reference" "R2202" (id 0) (at 101.854 67.4116 0)
@@
       (effects (font (size 1.524 1.524)))
     )
-    (property "PartNumber" "800235-301" (id 4) (at 104.902 66.04 90)
+    (property "PartNumber" "800235-XXX" (id 4) (at 104.902 66.04 90)
       (effects (font (size 1.524 1.524)) hide)
     )
@@
     (pin "2")
   )
-  (symbol (lib_id "Custom:R_US_0805_1%_HS") (at 116.84 68.58 0)
+  (symbol (lib_id "custom:R_US_0805_1%_HS") (at 116.84 68.58 0) (unit 1)
     (in_bom yes) (on_board yes)
     (property "Reference" "R2203" (id 0) (at 118.364 67.4116 0)
@@
       (effects (font (size 1.524 1.524)))
     )
-    (property "PartNumber" "800235-301" (id 4) (at 121.412 66.04 90)
+    (property "PartNumber" "800235-XXX" (id 4) (at 121.412 66.04 90)
       (effects (font (size 1.524 1.524)) hide)
     )
@@
     (pin "2")
   )
-  (symbol (lib_id "Custom:R_US_0805_1%_HS") (at 109.22 59.69 270)
+  (symbol (lib_id "custom:R_US_0805_1%_HS") (at 109.22 59.69 270) (unit 1)
     (in_bom yes) (on_board yes)
     (property "Reference" "R2201" (id 0) (at 109.22 54.6862 90))
@@
       (effects (font (size 1.524 1.524)))
     )
-    (property "PartNumber" "800235-180" (id 4) (at 111.76 64.262 90)
+    (property "PartNumber" "800235-XXX" (id 4) (at 111.76 64.262 90)
       (effects (font (size 1.524 1.524)) hide)
     )
@@
     (pin "2")
   )
-  (symbol (lib_id "Custom:GND_US") (at 100.33 73.66 0)
+  (symbol (lib_id "custom:GND_US") (at 100.33 73.66 0) (unit 1)
     (in_bom yes) (on_board yes)
     (property "Reference" "#PWR02201" (id 0) (at 99.822 76.962 0)
@@
     (pin "1")
   )
-  (symbol (lib_id "Custom:GND_US") (at 143.51 102.87 0)
+  (symbol (lib_id "custom:GND_US") (at 143.51 102.87 0) (unit 1)
     (in_bom yes) (on_board yes)
     (property "Reference" "#PWR02203" (id 0) (at 143.002 106.172 0)

Commit message: Fix BOM part number errors and out of sync footprints which happened during conversion from Kicad 5 to 6
Parts:
- R2201: PartNumber 800235-XXX -> 800235-180
- R2202, R2203: PartNumber 800235-XXX -> 800235-301
Changed lines of the file:
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@@
       (effects (font (size 1.524 1.524)))
     )
-    (property "PartNumber" "800235-XXX" (id 4) (at 104.902 66.04 90)
+    (property "PartNumber" "800235-301" (id 4) (at 104.902 66.04 90)
       (effects (font (size 1.524 1.524)) hide)
     )
@@
       (effects (font (size 1.524 1.524)))
     )
-    (property "PartNumber" "800235-XXX" (id 4) (at 121.412 66.04 90)
+    (property "PartNumber" "800235-301" (id 4) (at 121.412 66.04 90)
       (effects (font (size 1.524 1.524)) hide)
     )
@@
       (effects (font (size 1.524 1.524)))
     )
-    (property "PartNumber" "800235-XXX" (id 4) (at 111.76 64.262 90)
+    (property "PartNumber" "800235-180" (id 4) (at 111.76 64.262 90)
       (effects (font (size 1.524 1.524)) hide)
     )

Commit message: trx_mobo_concept_2_B. Change design to use a dedicated 8V supply for the 2SC3357 parts. Add S-Meter connector. Change mic connector to 3 pins and add 8V sopower supply to pin 3.
Parts:
- R1301: renamed from R2201; value 18 -> (none); footprint Resistor_SMD:R_0805_2012Metric_Pad1.15x1.40mm_HandSolder -> (none)
- R1302: renamed from R2202; value 300 -> (none); footprint Resistor_SMD:R_0805_2012Metric_Pad1.15x1.40mm_HandSolder -> (none)
- R1303: renamed from R2203; value 300 -> (none); footprint Resistor_SMD:R_0805_2012Metric_Pad1.15x1.40mm_HandSolder -> (none)
- U1301: renamed from U2201; value ADE-1 -> (none); footprint mods:MCL-6-SMD_7R97X5R59 -> (none)
Changed lines of the file:
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@@
   (title_block
     (title "THIRD_MIXER")
-    (rev "X1")
+    (rev "B")
   )
   (junction (at 100.33 59.69) (diameter 0) (color 0 0 0 0)
@@
   (symbol (lib_id "custom:ADE-1") (at 147.32 88.9 0) (unit 1)
     (in_bom yes) (on_board yes)
-    (property "Reference" "U2201" (id 0) (at 138.43 80.01 0)
-      (effects (font (size 1.27 1.27)) (justify left))
-    )
-    (property "Value" "ADE-1" (id 1) (at 149.86 81.28 0)
-      (effects (font (size 1.27 1.27)) (justify left))
-    )
-    (property "Footprint" "mods:MCL-6-SMD_7R97X5R59" (id 2) (at 147.32 88.9 0)
+    (property "Reference" "U1301" (id 0) (at 138.43 80.01 0)
+      (effects (font (size 1.27 1.27)) (justify left))
+    )
+    (property "Value" "" (id 1) (at 149.86 81.28 0)
+      (effects (font (size 1.27 1.27)) (justify left))
+    )
+    (property "Footprint" "" (id 2) (at 147.32 88.9 0)
       (effects (font (size 1.27 1.27)) hide)
     )
@@
   (symbol (lib_id "custom:GND_US") (at 116.84 73.66 0) (unit 1)
     (in_bom yes) (on_board yes)
-    (property "Reference" "#PWR02202" (id 0) (at 116.332 76.962 0)
+    (property "Reference" "#PWR01302" (id 0) (at 116.332 76.962 0)
       (effects (font (size 0.762 0.762)) hide)
     )
@@
   (symbol (lib_id "custom:GND_US") (at 147.32 102.87 0) (unit 1)
     (in_bom yes) (on_board yes)
-    (property "Reference" "#PWR02204" (id 0) (at 146.812 106.172 0)
+    (property "Reference" "#PWR01304" (id 0) (at 146.812 106.172 0)
       (effects (font (size 0.762 0.762)) hide)
     )
@@
   (symbol (lib_id "custom:GND_US") (at 151.13 102.87 0) (unit 1)
     (in_bom yes) (on_board yes)
-    (property "Reference" "#PWR02205" (id 0) (at 150.622 106.172 0)
+    (property "Reference" "#PWR01305" (id 0) (at 150.622 106.172 0)
       (effects (font (size 0.762 0.762)) hide)
     )
@@
   (symbol (lib_id "custom:R_US_0805_1%_HS") (at 100.33 68.58 0) (unit 1)
     (in_bom yes) (on_board yes)
-    (property "Reference" "R2202" (id 0) (at 101.854 67.4116 0)
-      (effects (font (size 1.27 1.27)) (justify left))
-    )
-    (property "Value" "300" (id 1) (at 101.854 69.723 0)
-      (effects (font (size 1.27 1.27)) (justify left))
-    )
-    (property "Footprint" "Resistor_SMD:R_0805_2012Metric_Pad1.15x1.40mm_HandSolder" (id 2) (at 100.33 68.58 0)
+    (property "Reference" "R1302" (id 0) (at 101.854 67.4116 0)
+      (effects (font (size 1.27 1.27)) (justify left))
+    )
+    (property "Value" "" (id 1) (at 101.854 69.723 0)
+      (effects (font (size 1.27 1.27)) (justify left))
+    )
+    (property "Footprint" "" (id 2) (at 100.33 68.58 0)
       (effects (font (size 1.524 1.524)) hide)
     )
@@
   (symbol (lib_id "custom:R_US_0805_1%_HS") (at 116.84 68.58 0) (unit 1)
     (in_bom yes) (on_board yes)
-    (property "Reference" "R2203" (id 0) (at 118.364 67.4116 0)
-      (effects (font (size 1.27 1.27)) (justify left))
-    )
-    (property "Value" "300" (id 1) (at 118.364 69.723 0)
-      (effects (font (size 1.27 1.27)) (justify left))
-    )
-    (property "Footprint" "Resistor_SMD:R_0805_2012Metric_Pad1.15x1.40mm_HandSolder" (id 2) (at 116.84 68.58 0)
+    (property "Reference" "R1303" (id 0) (at 118.364 67.4116 0)
+      (effects (font (size 1.27 1.27)) (justify left))
+    )
+    (property "Value" "" (id 1) (at 118.364 69.723 0)
+      (effects (font (size 1.27 1.27)) (justify left))
+    )
+    (property "Footprint" "" (id 2) (at 116.84 68.58 0)
       (effects (font (size 1.524 1.524)) hide)
     )
@@
   (symbol (lib_id "custom:R_US_0805_1%_HS") (at 109.22 59.69 270) (unit 1)
     (in_bom yes) (on_board yes)
-    (property "Reference" "R2201" (id 0) (at 109.22 54.6862 90))
-    (property "Value" "18" (id 1) (at 109.22 56.9976 90))
-    (property "Footprint" "Resistor_SMD:R_0805_2012Metric_Pad1.15x1.40mm_HandSolder" (id 2) (at 109.22 59.69 0)
+    (property "Reference" "R1301" (id 0) (at 109.22 54.6862 90))
+    (property "Value" "" (id 1) (at 109.22 56.9976 90))
+    (property "Footprint" "" (id 2) (at 109.22 59.69 0)
       (effects (font (size 1.524 1.524)) hide)
     )
@@
   (symbol (lib_id "custom:GND_US") (at 100.33 73.66 0) (unit 1)
     (in_bom yes) (on_board yes)
-    (property "Reference" "#PWR02201" (id 0) (at 99.822 76.962 0)
+    (property "Reference" "#PWR01301" (id 0) (at 99.822 76.962 0)
       (effects (font (size 0.762 0.762)) hide)
     )
@@
   (symbol (lib_id "custom:GND_US") (at 143.51 102.87 0) (unit 1)
     (in_bom yes) (on_board yes)
-    (property "Reference" "#PWR02203" (id 0) (at 143.002 106.172 0)
-      (effects (font (size 0.762 0.762)) hide)
-    )
+    (property "Reference" "#PWR01303" (id 0) (at 143.002 106.172 0)
+      (effects (font (size 0.762 0.762)) hide)
+    )
