File: i2c.kicad_sch (KiCad schematic)
At the start: 14 parts, among them Q401 BSS138, Q402 BSS138, U401 24CW640, U402 MCP4725, U403 74LVC1G00

Commit message: Update pcb database to version 6
Parts:
- C401, C402, C403: symbol Custom:C_US_0805_0.1UF_X7R_10%_50V_HS -> custom:C_US_0805_0.1UF_X7R_10%_50V_HS
- C404: symbol Custom:C_US_0805_0.1UF_X7R_10%_50V_HS -> custom:C_US_0805_0.1UF_X7R_10%_50V_HS; PartNumber 800238-105 -> 800238-104
- C405: footprint Capacitor_SMD:C_0805_2012Metric_Pad1.15x1.40mm_HandSolder -> Capacitor_SMD:C_0603_1608Metric; symbol Custom:C_US -> custom:C_US; PartNumber 800003-106 -> 800063-XXX
- Q401, Q402: footprint mods:SOT23-3-SAR -> SOT-23; symbol Custom:BSS138 -> custom:BSS138
- R401, R402: symbol Custom:R_US_0805_1%_HS -> custom:R_US_0805_1%_HS; PartNumber 800235-103 -> 800235-XXX
- R403: symbol Custom:R_US_0805_1%_HS -> custom:R_US_0805_1%_HS; PartNumber 800235-101 -> 800235-XXX
- U401: symbol Custom:24CW640 -> custom:24CW640
- U402: footprint mods:SOT23-6-SAR -> mods:SOT23-5-SAR; symbol Custom:MCP4725 -> custom:MCP4725
- U403: symbol Custom:74LVC1G00 -> custom:74LVC1G00
- VR401: footprint mods:SOT23-3-SAR -> SOT23-3; symbol Custom:ME6211A33M3G-N -> custom:ME6211A33M3G-N

Commit message: Sync PCB with schematic
Parts:
- C405: footprint Capacitor_SMD:C_0603_1608Metric -> Capacitor_SMD:C_0805_2012Metric_Pad1.15x1.40mm_HandSolder
- Q401, Q402: footprint SOT-23 -> mods:SOT23-3-SAR
- U402: footprint mods:SOT23-5-SAR -> mods:SOT23-6-SAR
- VR401: footprint SOT23-3 -> mods:SOT23-3-SAR
Changed lines of the file:
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@@
       (effects (font (size 1.27 1.27)) (justify left))
     )
-    (property "Footprint" "Capacitor_SMD:C_0603_1608Metric" (id 2) (at 128.27 162.56 0)
+    (property "Footprint" "Capacitor_SMD:C_0805_2012Metric_Pad1.15x1.40mm_HandSolder" (id 2) (at 128.27 162.56 0)
       (effects (font (size 1.524 1.524)) hide)
     )
@@
     (property "Reference" "VR401" (id 0) (at 73.66 155.829 0))
     (property "Value" "ME6211A33M3G-N" (id 1) (at 73.66 158.1404 0))
-    (property "Footprint" "SOT23-3" (id 2) (at 73.66 161.29 0)
+    (property "Footprint" "mods:SOT23-3-SAR" (id 2) (at 73.66 161.29 0)
       (effects (font (size 1.27 1.27)) hide)
     )
@@
       (effects (font (size 1.016 1.016)))
     )
-    (property "Footprint" "SOT-23" (id 2) (at 58.4708 108.458 0)
+    (property "Footprint" "mods:SOT23-3-SAR" (id 2) (at 58.4708 108.458 0)
       (effects (font (size 0.7366 0.7366)) hide)
     )
@@
       (effects (font (size 1.016 1.016)))
     )
-    (property "Footprint" "SOT-23" (id 2) (at 58.4708 131.318 0)
+    (property "Footprint" "mods:SOT23-3-SAR" (id 2) (at 58.4708 131.318 0)
       (effects (font (size 0.7366 0.7366)) hide)
     )
@@
       (effects (font (size 1.27 1.27)) (justify left))
     )
-    (property "Footprint" "mods:SOT23-5-SAR" (id 2) (at 146.05 134.62 0)
-      (effects (font (size 1.524 1.524)) hide)
-    )
+    (property "Footprint" "mods:SOT23-6-SAR" (id 2) (at 146.05 134.62 0)
+      (effects (font (size 1.524 1.524)) hide)
+    )

Commit message: Fix BOM part number errors and out of sync footprints which happened during conversion from Kicad 5 to 6
Parts:
- C404: PartNumber 800238-104 -> 800238-105
- C405: PartNumber 800063-XXX -> 800003-106
- R401, R402: PartNumber 800235-XXX -> 800235-103
- R403: PartNumber 800235-XXX -> 800235-101
Changed lines of the file:
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@@
       (effects (font (size 1.524 1.524)))
     )
-    (property "PartNumber" "800063-XXX" (id 4) (at 125.73 160.02 0)
+    (property "PartNumber" "800003-106" (id 4) (at 125.73 160.02 0)
       (effects (font (size 1.524 1.524)) hide)
     )
@@
       (effects (font (size 1.524 1.524)))
     )
-    (property "PartNumber" "800238-104" (id 4) (at 49.53 158.75 0)
+    (property "PartNumber" "800238-105" (id 4) (at 49.53 158.75 0)
       (effects (font (size 1.524 1.524)) hide)
     )
@@
       (effects (font (size 1.524 1.524)))
     )
-    (property "PartNumber" "800235-XXX" (id 4) (at 73.152 99.06 90)
+    (property "PartNumber" "800235-103" (id 4) (at 73.152 99.06 90)
       (effects (font (size 1.524 1.524)) hide)
     )
@@
       (effects (font (size 1.524 1.524)))
     )
-    (property "PartNumber" "800235-XXX" (id 4) (at 84.582 99.06 90)
+    (property "PartNumber" "800235-103" (id 4) (at 84.582 99.06 90)
       (effects (font (size 1.524 1.524)) hide)
     )
@@
       (effects (font (size 1.524 1.524)))
     )
-    (property "PartNumber" "800235-XXX" (id 4) (at 168.91 129.032 90)
-      (effects (font (size 1.524 1.524)) hide)
-    )
+    (property "PartNumber" "800235-101" (id 4) (at 168.91 129.032 90)
+      (effects (font (size 1.524 1.524)) hide)
+    )

Commit message: trx_mobo_concept_2_B. Change design to use a dedicated 8V supply for the 2SC3357 parts. Add S-Meter connector. Change mic connector to 3 pins and add 8V sopower supply to pin 3.
Parts:
- C301: renamed from C401; value 0.1u -> (none); footprint Capacitor_SMD:C_0805_2012Metric_Pad1.15x1.40mm_HandSolder -> (none)
- C302: renamed from C402; value 0.1u -> (none); footprint Capacitor_SMD:C_0805_2012Metric_Pad1.15x1.40mm_HandSolder -> (none)
- C303: renamed from C403; value 0.1u -> (none); footprint Capacitor_SMD:C_0805_2012Metric_Pad1.15x1.40mm_HandSolder -> (none)
- C304: renamed from C404; value 1u -> (none); footprint Capacitor_SMD:C_0805_2012Metric_Pad1.15x1.40mm_HandSolder -> (none)
- C305: renamed from C405; value 10u -> (none); footprint Capacitor_SMD:C_0805_2012Metric_Pad1.15x1.40mm_HandSolder -> (none)
- Q301: renamed from Q401; value BSS138 -> (none); footprint mods:SOT23-3-SAR -> (none)
- Q302: renamed from Q402; value BSS138 -> (none); footprint mods:SOT23-3-SAR -> (none)
- R301: renamed from R401; value 10K -> (none); footprint Resistor_SMD:R_0805_2012Metric_Pad1.15x1.40mm_HandSolder -> (none)
- R302: renamed from R402; value 10K -> (none); footprint Resistor_SMD:R_0805_2012Metric_Pad1.15x1.40mm_HandSolder -> (none)
- R303: renamed from R403; value 100 -> (none); footprint Resistor_SMD:R_0805_2012Metric_Pad1.15x1.40mm_HandSolder -> (none)
- U301: renamed from U401; value 24CW640 -> (none); footprint mods:SOT23-5-SAR -> (none)
- U302: renamed from U402; value MCP4725 -> (none); footprint mods:SOT23-6-SAR -> (none)
- U303: renamed from U403; value 74LVC1G00 -> (none); footprint mods:SOT23-5-SAR -> (none)
- VR301: renamed from VR401; value ME6211A33M3G-N -> (none); footprint mods:SOT23-3-SAR -> (none)
