File: radio.kicad_sch (KiCad schematic)
At the start: 0 parts

Commit message: trx_mobo_concept_2_B. Change design to use a dedicated 8V supply for the 2SC3357 parts. Add S-Meter connector. Change mic connector to 3 pins and add 8V sopower supply to pin 3.
Other:
- sheet prod_det_tx_mix ports: added S_METER; removed none
- sheet rf_45r1_mic_amp_tune_osc ports: added P8V0_TX; removed none
Changed lines of the file:
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@@
   (paper "A4")
   (title_block
-    (rev "X1")
+    (rev "B")
     (company "WA6ZFT")
   )
@@
     (stroke (width 0) (type default) (color 0 0 0 0))
   )
+  (wire (pts (xy 130.81 162.56) (xy 130.81 157.48))
+    (stroke (width 0) (type default) (color 0 0 0 0))
+  )
   (wire (pts (xy 190.5 147.32) (xy 267.97 147.32))
     (stroke (width 0) (type default) (color 0 0 0 0))
@@
     (stroke (width 0) (type default) (color 0 0 0 0))
   )
+  (wire (pts (xy 73.66 162.56) (xy 130.81 162.56))
+    (stroke (width 0) (type default) (color 0 0 0 0))
+  )
   (wire (pts (xy 38.1 140.97) (xy 38.1 73.66))
     (stroke (width 0) (type default) (color 0 0 0 0))
@@
     (stroke (width 0) (type default) (color 0 0 0 0))
   )
+  (wire (pts (xy 130.81 157.48) (xy 267.97 157.48))
+    (stroke (width 0) (type default) (color 0 0 0 0))
+  )
   (wire (pts (xy 29.21 58.42) (xy 205.74 58.42))
     (stroke (width 0) (type default) (color 0 0 0 0))
@@
   )
   (wire (pts (xy 39.37 166.37) (xy 48.26 166.37))
+    (stroke (width 0) (type default) (color 0 0 0 0))
+  )
+  (wire (pts (xy 256.54 116.84) (xy 267.97 116.84))
     (stroke (width 0) (type default) (color 0 0 0 0))
   )
@@
     (effects (font (size 1.27 1.27)) (justify left))
   )
+  (hierarchical_label "S_METER" (shape passive) (at 267.97 116.84 0)
+    (effects (font (size 1.27 1.27)) (justify left))
+  )
   (hierarchical_label "MUTE_RX_AUDIO" (shape input) (at 29.21 38.1 180)
     (effects (font (size 1.27 1.27)) (justify right))
@@
   (hierarchical_label "TX_AUDIO_IN" (shape passive) (at 33.02 162.56 180)
     (effects (font (size 1.27 1.27)) (justify right))
+  )
+  (hierarchical_label "P8V0_TX" (shape passive) (at 267.97 157.48 0)
+    (effects (font (size 1.27 1.27)) (justify left))
   )
   (hierarchical_label "TX_IF_GAIN" (shape passive) (at 29.21 33.02 180)
@@
       (effects (font (size 1.27 1.27)) (justify left))
     )
+    (pin "P8V0_TX" passive (at 73.66 162.56 0)
+      (effects (font (size 1.27 1.27)) (justify right))
+    )
   )
   (sheet (at 124.46 88.9) (size 12.7 24.13) (fields_autoplaced)
@@
     )
   )
-  (sheet (at 167.64 88.9) (size 16.51 24.13) (fields_autoplaced)
+  (sheet (at 167.64 88.9) (size 16.51 24.13)
     (stroke (width 0) (type solid) (color 0 0 0 0))
     (fill (color 0 0 0 0.0000))
@@
       (effects (font (size 1.27 1.27)) (justify left bottom))
     )
-    (property "Sheet file" "ifagc.kicad_sch" (id 1) (at 167.64 113.6146 0)
+    (property "Sheet file" "ifagc.kicad_sch" (id 1) (at 162.56 113.03 0)
       (effects (font (size 1.27 1.27)) (justify left top))
     )
@@
       (effects (font (size 1.27 1.27)) (justify left))
     )
-  )
+    (pin "S_METER" passive (at 256.54 116.84 0)
+      (effects (font (size 1.27 1.27)) (justify right))
+    )
+  )
