File: xtal_filter.kicad_sch (KiCad schematic)
At the start: 30 parts, among them Y701 12.288 MHz, Y702 12.288 MHz, Y703 12.288 MHz, Y704 12.288 MHz, Y705 12.288 MHz, Y706 12.288 MHz

Commit message: Update pcb database to version 6
Parts:
- C701, C702: symbol Custom:C_US_0805_C0G_NPO_5%_50V_HS -> custom:C_US_0805_C0G_NPO_5%_50V_HS; PartNumber 800239-431 -> 800239_XXX
- C703, C704: symbol Custom:C_US_0805_C0G_NPO_5%_50V_HS -> custom:C_US_0805_C0G_NPO_5%_50V_HS; PartNumber 800239-150 -> 800239_XXX
- C705, C710: symbol Custom:C_US_0805_C0G_NPO_5%_50V_HS -> custom:C_US_0805_C0G_NPO_5%_50V_HS; PartNumber 800239-121 -> 800239_XXX
- C706, C709, C712, C713, C716, C717, C719: symbol Custom:C_US_0805_C0G_NPO_5%_50V_HS -> custom:C_US_0805_C0G_NPO_5%_50V_HS; PartNumber 800239-151 -> 800239_XXX
- C707, C708, C714, C715: symbol Custom:C_US_0805_C0G_NPO_5%_50V_HS -> custom:C_US_0805_C0G_NPO_5%_50V_HS; PartNumber 800239-100 -> 800239_XXX
- C711: symbol Custom:C_US_0805_C0G_NPO_5%_50V_HS -> custom:C_US_0805_C0G_NPO_5%_50V_HS; PartNumber 800239-180 -> 800239_XXX
- C718, C720: symbol Custom:C_US_0805_C0G_NPO_5%_50V_HS -> custom:C_US_0805_C0G_NPO_5%_50V_HS; PartNumber 800239-200 -> 800239_XXX
- R701, R702: symbol Custom:R_US -> custom:R_US; PartNumber 800235-000 -> 800XXX-XXX
- Y701, Y702, Y703, Y704, Y705, Y706: symbol Custom:Crystal_with_GND -> custom:Crystal_with_GND; PartNumber 800286-101 -> 800260-101

Commit message: Fix BOM part number errors and out of sync footprints which happened during conversion from Kicad 5 to 6
Parts:
- C701, C702: PartNumber 800239_XXX -> 800239-431
- C703, C704: PartNumber 800239_XXX -> 800239-150
- C705, C710: PartNumber 800239_XXX -> 800239-121
- C706, C709, C712, C713, C716, C717, C719: PartNumber 800239_XXX -> 800239-151
- C707, C708, C714, C715: PartNumber 800239_XXX -> 800239-100
- C711: PartNumber 800239_XXX -> 800239-180
- C718, C720: PartNumber 800239_XXX -> 800239-200
- R701, R702: PartNumber 800XXX-XXX -> 800235-000
Changed lines of the file:
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@@
       (effects (font (size 1.524 1.524)))
     )
-    (property "PartNumber" "800239_XXX" (id 4) (at 232.41 26.67 0)
+    (property "PartNumber" "800239-121" (id 4) (at 232.41 26.67 0)
       (effects (font (size 1.524 1.524)) hide)
     )
@@
       (effects (font (size 1.524 1.524)))
     )
-    (property "PartNumber" "800239_XXX" (id 4) (at 63.5 26.67 0)
+    (property "PartNumber" "800239-121" (id 4) (at 63.5 26.67 0)
       (effects (font (size 1.524 1.524)) hide)
     )
@@
       (effects (font (size 1.524 1.524)))
     )
-    (property "PartNumber" "800239_XXX" (id 4) (at 91.44 26.67 0)
+    (property "PartNumber" "800239-151" (id 4) (at 91.44 26.67 0)
       (effects (font (size 1.524 1.524)) hide)
     )
@@
       (effects (font (size 1.524 1.524)))
     )
-    (property "PartNumber" "800239_XXX" (id 4) (at 203.2 26.67 0)
+    (property "PartNumber" "800239-151" (id 4) (at 203.2 26.67 0)
       (effects (font (size 1.524 1.524)) hide)
     )
@@
       (effects (font (size 1.524 1.524)))
     )
-    (property "PartNumber" "800239_XXX" (id 4) (at 149.86 25.4 0)
+    (property "PartNumber" "800239-431" (id 4) (at 149.86 25.4 0)
       (effects (font (size 1.524 1.524)) hide)
     )
@@
       (effects (font (size 1.524 1.524)))
     )
-    (property "PartNumber" "800239_XXX" (id 4) (at 102.87 26.67 0)
+    (property "PartNumber" "800239-100" (id 4) (at 102.87 26.67 0)
       (effects (font (size 1.524 1.524)) hide)
     )
@@
       (effects (font (size 1.524 1.524)))
     )
-    (property "PartNumber" "800239_XXX" (id 4) (at 193.04 26.67 0)
+    (property "PartNumber" "800239-100" (id 4) (at 193.04 26.67 0)
       (effects (font (size 1.524 1.524)) hide)
     )
@@
       (effects (font (size 1.524 1.524)))
     )
-    (property "PartNumber" "800239_XXX" (id 4) (at 25.4 54.61 0)
+    (property "PartNumber" "800239-151" (id 4) (at 25.4 54.61 0)
       (effects (font (size 1.524 1.524)) hide)
     )
@@
       (effects (font (size 1.524 1.524)))
     )
-    (property "PartNumber" "800239_XXX" (id 4) (at 38.1 54.61 0)
+    (property "PartNumber" "800239-100" (id 4) (at 38.1 54.61 0)
       (effects (font (size 1.524 1.524)) hide)
     )
@@
       (effects (font (size 1.524 1.524)))
     )
-    (property "PartNumber" "800239_XXX" (id 4) (at 257.81 57.15 0)
+    (property "PartNumber" "800239-151" (id 4) (at 257.81 57.15 0)
       (effects (font (size 1.524 1.524)) hide)
     )
@@
       (effects (font (size 1.524 1.524)))
     )
-    (property "PartNumber" "800239_XXX" (id 4) (at 246.38 57.15 0)
+    (property "PartNumber" "800239-100" (id 4) (at 246.38 57.15 0)
       (effects (font (size 1.524 1.524)) hide)
     )
@@
       (effects (font (size 1.524 1.524)))
     )
-    (property "PartNumber" "800239_XXX" (id 4) (at 172.72 25.4 0)
+    (property "PartNumber" "800239-431" (id 4) (at 172.72 25.4 0)
       (effects (font (size 1.524 1.524)) hide)
     )
@@
       (effects (font (size 1.524 1.524)))
     )
-    (property "PartNumber" "800239_XXX" (id 4) (at 149.86 36.83 0)
+    (property "PartNumber" "800239-150" (id 4) (at 149.86 36.83 0)
       (effects (font (size 1.524 1.524)) hide)
     )
@@
       (effects (font (size 1.524 1.524)))
     )
-    (property "PartNumber" "800239_XXX" (id 4) (at 172.72 36.83 0)
+    (property "PartNumber" "800239-150" (id 4) (at 172.72 36.83 0)
       (effects (font (size 1.524 1.524)) hide)
     )
@@
       (effects (font (size 1.524 1.524)))
     )
-    (property "PartNumber" "800239_XXX" (id 4) (at 25.4 96.52 0)
+    (property "PartNumber" "800239-151" (id 4) (at 25.4 96.52 0)
       (effects (font (size 1.524 1.524)) hide)
     )
@@
       (effects (font (size 1.524 1.524)))
     )
-    (property "PartNumber" "800239_XXX" (id 4) (at 38.1 96.52 0)
+    (property "PartNumber" "800239-200" (id 4) (at 38.1 96.52 0)
       (effects (font (size 1.524 1.524)) hide)
     )
@@
       (effects (font (size 1.524 1.524)))
     )
-    (property "PartNumber" "800239_XXX" (id 4) (at 246.38 93.98 0)
+    (property "PartNumber" "800239-151" (id 4) (at 246.38 93.98 0)
       (effects (font (size 1.524 1.524)) hide)
     )
@@
       (effects (font (size 1.524 1.524)))
     )
-    (property "PartNumber" "800239_XXX" (id 4) (at 257.81 93.98 0)
+    (property "PartNumber" "800239-200" (id 4) (at 257.81 93.98 0)
       (effects (font (size 1.524 1.524)) hide)
     )
@@
       (effects (font (size 1.524 1.524)))
     )
-    (property "PartNumber" "800XXX-XXX" (id 4) (at 53.34 96.012 90)
+    (property "PartNumber" "800235-000" (id 4) (at 53.34 96.012 90)
       (effects (font (size 1.524 1.524)) hide)
     )
@@
       (effects (font (size 1.524 1.524)))
     )
-    (property "PartNumber" "800XXX-XXX" (id 4) (at 233.68 94.742 90)
+    (property "PartNumber" "800235-000" (id 4) (at 233.68 94.742 90)
       (effects (font (size 1.524 1.524)) hide)
     )
@@
       (effects (font (size 1.524 1.524)))
     )
-    (property "PartNumber" "800239_XXX" (id 4) (at 152.4 41.91 0)
+    (property "PartNumber" "800239-151" (id 4) (at 152.4 41.91 0)
       (effects (font (size 1.524 1.524)) hide)
     )
@@
       (effects (font (size 1.524 1.524)))
     )
-    (property "PartNumber" "800239_XXX" (id 4) (at 140.97 41.91 0)
-      (effects (font (size 1.524 1.524)) hide)
-    )
+    (property "PartNumber" "800239-180" (id 4) (at 140.97 41.91 0)
+      (effects (font (size 1.524 1.524)) hide)
+    )

Commit message: trx_mobo_concept_2_B. Change design to use a dedicated 8V supply for the 2SC3357 parts. Add S-Meter connector. Change mic connector to 3 pins and add 8V sopower supply to pin 3.
Parts:
- C1701: renamed from C701; value 430p -> (none); footprint Capacitor_SMD:C_0805_2012Metric_Pad1.15x1.40mm_HandSolder -> (none)
- C1702: renamed from C702; value 430p -> (none); footprint Capacitor_SMD:C_0805_2012Metric_Pad1.15x1.40mm_HandSolder -> (none)
- C1703: renamed from C703; value 15p -> (none); footprint Capacitor_SMD:C_0805_2012Metric_Pad1.15x1.40mm_HandSolder -> (none)
- C1704: renamed from C704; value 15p -> (none); footprint Capacitor_SMD:C_0805_2012Metric_Pad1.15x1.40mm_HandSolder -> (none)
- C1705: renamed from C705; value 120p -> (none); footprint Capacitor_SMD:C_0805_2012Metric_Pad1.15x1.40mm_HandSolder -> (none)
- C1706: renamed from C706; value 150p -> (none); footprint Capacitor_SMD:C_0805_2012Metric_Pad1.15x1.40mm_HandSolder -> (none)
- C1707: renamed from C707; value 10p -> (none); footprint Capacitor_SMD:C_0805_2012Metric_Pad1.15x1.40mm_HandSolder -> (none)
- C1708: renamed from C708; value 10p -> (none); footprint Capacitor_SMD:C_0805_2012Metric_Pad1.15x1.40mm_HandSolder -> (none)
- C1709: renamed from C709; value 150P -> (none); footprint Capacitor_SMD:C_0805_2012Metric_Pad1.15x1.40mm_HandSolder -> (none)
- C1710: renamed from C710; value 120p -> (none); footprint Capacitor_SMD:C_0805_2012Metric_Pad1.15x1.40mm_HandSolder -> (none)
- C1711: renamed from C711; value 18p -> (none); footprint Capacitor_SMD:C_0805_2012Metric_Pad1.15x1.40mm_HandSolder -> (none)
- C1712: renamed from C712; value 150p -> (none); footprint Capacitor_SMD:C_0805_2012Metric_Pad1.15x1.40mm_HandSolder -> (none)
- C1713: renamed from C713; value 150p -> (none); footprint Capacitor_SMD:C_0805_2012Metric_Pad1.15x1.40mm_HandSolder -> (none)
- C1714: renamed from C714; value 10p -> (none); footprint Capacitor_SMD:C_0805_2012Metric_Pad1.15x1.40mm_HandSolder -> (none)
- C1715: renamed from C715; value 10p -> (none); footprint Capacitor_SMD:C_0805_2012Metric_Pad1.15x1.40mm_HandSolder -> (none)
- C1716: renamed from C716; value 150P -> (none); footprint Capacitor_SMD:C_0805_2012Metric_Pad1.15x1.40mm_HandSolder -> (none)
- C1717: renamed from C717; value 150p -> (none); footprint Capacitor_SMD:C_0805_2012Metric_Pad1.15x1.40mm_HandSolder -> (none)
- C1718: renamed from C718; value 20p -> (none); footprint Capacitor_SMD:C_0805_2012Metric_Pad1.15x1.40mm_HandSolder -> (none)
- C1719: renamed from C719; value 150p -> (none); footprint Capacitor_SMD:C_0805_2012Metric_Pad1.15x1.40mm_HandSolder -> (none)
- C1720: renamed from C720; value 20p -> (none); footprint Capacitor_SMD:C_0805_2012Metric_Pad1.15x1.40mm_HandSolder -> (none)
- L1701: renamed from L701; value 0.97uH -> (none); footprint mods:TOROID_T37_VERT -> (none)
- L1702: renamed from L702; value 0.97uH -> (none); footprint mods:TOROID_T37_VERT -> (none)
- R1701: renamed from R701; value 0 -> (none); footprint Resistor_SMD:R_0805_2012Metric_Pad1.15x1.40mm_HandSolder -> (none)
- R1702: renamed from R702; value 0 -> (none); footprint Resistor_SMD:R_0805_2012Metric_Pad1.15x1.40mm_HandSolder -> (none)
- Y1701: renamed from Y701; value 12.288 MHz -> (none); footprint mods:Crystal_HC49_Vertical_With_Grounding_Pad -> (none)
- Y1702: renamed from Y702; value 12.288 MHz -> (none); footprint mods:Crystal_HC49_Vertical_With_Grounding_Pad -> (none)
- Y1703: renamed from Y703; value 12.288 MHz -> (none); footprint mods:Crystal_HC49_Vertical_With_Grounding_Pad -> (none)
- Y1704: renamed from Y704; value 12.288 MHz -> (none); footprint mods:Crystal_HC49_Vertical_With_Grounding_Pad -> (none)
- Y1705: renamed from Y705; value 12.288 MHz -> (none); footprint mods:Crystal_HC49_Vertical_With_Grounding_Pad -> (none)
- Y1706: renamed from Y706; value 12.288 MHz -> (none); footprint mods:Crystal_HC49_Vertical_With_Grounding_Pad -> (none)
Other:
- note added: "16T #28 AWG T37-6"
- note removed: "-6dB lower: 12.284950 MHz"
- note removed: "-6db upper: 12.287500 MHz"
- note removed: "16T #28 AWG"
- note removed: "Center Freq: 12.286225 MHz"
- note removed: "Loss: 3.67db"
- note removed: "Measured -6dB BW: 2550 Hz"
- note removed: "SN #1 Measurements"

Commit message: Fix 12.288MHz part number in schematic, regenerate BOM's.
Parts:
- Y1701, Y1702, Y1703, Y1704, Y1705, Y1706: PartNumber 800260-101 -> 800286-101
Changed lines of the file:
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@@
       (effects (font (size 1.27 1.27)) hide)
     )
-    (property "PartNumber" "800260-101" (id 4) (at 44.45 33.02 0)
+    (property "PartNumber" "800286-101" (id 4) (at 44.45 33.02 0)
       (effects (font (size 1.27 1.27)) hide)
     )
@@
       (effects (font (size 1.27 1.27)) hide)
     )
-    (property "PartNumber" "800260-101" (id 4) (at 82.55 33.02 0)
+    (property "PartNumber" "800286-101" (id 4) (at 82.55 33.02 0)
       (effects (font (size 1.27 1.27)) hide)
     )
@@
       (effects (font (size 1.27 1.27)) hide)
     )
-    (property "PartNumber" "800260-101" (id 4) (at 120.65 33.02 0)
+    (property "PartNumber" "800286-101" (id 4) (at 120.65 33.02 0)
       (effects (font (size 1.27 1.27)) hide)
     )
@@
       (effects (font (size 1.27 1.27)) hide)
     )
-    (property "PartNumber" "800260-101" (id 4) (at 177.8 33.02 0)
+    (property "PartNumber" "800286-101" (id 4) (at 177.8 33.02 0)
       (effects (font (size 1.27 1.27)) hide)
     )
@@
       (effects (font (size 1.27 1.27)) hide)
     )
-    (property "PartNumber" "800260-101" (id 4) (at 219.71 33.02 0)
+    (property "PartNumber" "800286-101" (id 4) (at 219.71 33.02 0)
       (effects (font (size 1.27 1.27)) hide)
     )
@@
       (effects (font (size 1.27 1.27)) hide)
     )
-    (property "PartNumber" "800260-101" (id 4) (at 247.65 33.02 0)
+    (property "PartNumber" "800286-101" (id 4) (at 247.65 33.02 0)
       (effects (font (size 1.27 1.27)) hide)
     )
